File: CAD/driver/clock_driver_board.brd (EAGLE design)
At the start: 61 x 40.4 mm, 21 parts, among them U1 MIC5891, U2 MIC5891, U3 HEX_CONVERTERDIP16

Commit message: Updated driver board CAD files for BOM
Parts:
- R1: value 500Ohm -> 470Ohm
Changed lines of the file:
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@@
 <element name="C2" library="capacitor-wima" package="C2.5-2" value="0.1uF" x="34.163" y="30.099" smashed="yes" rot="R180">
 <attribute name="VALUE" x="35.814" y="32.893" size="1.27" layer="27" ratio="10" rot="R180"/>
+<attribute name="PARTNO" value="21RZ310-RC" x="34.163" y="30.099" size="1.778" layer="27" rot="R180" display="off"/>
 </element>
 <element name="C1" library="capacitor-wima" package="C2.5-2" value="0.1uF" x="21.717" y="11.049" smashed="yes">
 <attribute name="VALUE" x="20.066" y="8.255" size="1.27" layer="27" ratio="10"/>
+<attribute name="PARTNO" value="21RZ310-RC" x="21.717" y="11.049" size="1.778" layer="27" display="off"/>
 </element>
 <element name="C3" library="capacitor-wima" package="C2.5-2" value="0.1uF" x="47.752" y="30.099" smashed="yes">
 <attribute name="VALUE" x="46.101" y="27.305" size="1.27" layer="27" ratio="10"/>
+<attribute name="PARTNO" value="21RZ310-RC" x="47.752" y="30.099" size="1.778" layer="27" display="off"/>
 </element>
 <element name="P8" library="SparkFun-Connectors" package="1X04_LONGPADS" value="" x="3.81" y="18.415" smashed="yes" rot="R90">
 <attribute name="VALUE" x="7.62" y="17.145" size="1.27" layer="27" rot="R90"/>
+<attribute name="PARTNO" value="826631-4" x="3.81" y="18.415" size="1.778" layer="27" rot="R90" display="off"/>
 </element>
 <element name="P0" library="SparkFun-Connectors" package="1X03_LONGPADS" value="" x="44.45" y="38.1" smashed="yes">
 <attribute name="NAME" x="45.6438" y="34.7218" size="1.016" layer="21" font="vector" ratio="10"/>
 <attribute name="VALUE" x="43.18" y="34.29" size="1.27" layer="27"/>
+<attribute name="BOM" value="EXCLUDE" x="44.45" y="38.1" size="1.778" layer="27" display="off"/>
 </element>
 <element name="P10" library="SparkFun-Connectors" package="SCREWTERMINAL-3.5MM-3" value="" x="3.81" y="36.83" smashed="yes" rot="R270">
 <attribute name="PROD_ID" value="CONN-08288" x="3.81" y="36.83" size="1.778" layer="27" rot="R270" display="off"/>
 <attribute name="VALUE" x="5.08" y="38.1" size="0.4064" layer="27" rot="R270"/>
+<attribute name="PARTNO" value="1546551-3" x="3.81" y="36.83" size="1.778" layer="27" rot="R270" display="off"/>
 </element>
 <element name="P11" library="SparkFun-Connectors" package="SCREWTERMINAL-3.5MM-3" value="" x="57.15" y="29.845" smashed="yes" rot="R90">
 <attribute name="PROD_ID" value="CONN-08288" x="57.15" y="29.845" size="1.778" layer="27" rot="R90" display="off"/>
 <attribute name="VALUE" x="55.88" y="28.575" size="0.4064" layer="27" rot="R90"/>
+<attribute name="PARTNO" value="1546551-3" x="57.15" y="29.845" size="1.778" layer="27" rot="R90" display="off"/>
 </element>
 <element name="P7" library="SparkFun-Connectors" package="1X03_LONGPADS" value="" x="49.53" y="3.81" smashed="yes" rot="R180">
 <attribute name="NAME" x="48.8442" y="7.0612" size="1.016" layer="21" font="vector" ratio="10" rot="R180"/>
 <attribute name="VALUE" x="50.8" y="7.62" size="1.27" layer="27" rot="R180"/>
+<attribute name="BOM" value="EXCLUDE" x="49.53" y="3.81" size="1.778" layer="27" rot="R180" display="off"/>
 </element>
 <element name="P6" library="SparkFun-Connectors" package="1X03_LONGPADS" value="" x="40.64" y="3.81" smashed="yes" rot="R180">
 <attribute name="NAME" x="39.4462" y="7.0612" size="1.016" layer="21" font="vector" ratio="10" rot="R180"/>
 <attribute name="VALUE" x="41.91" y="7.62" size="1.27" layer="27" rot="R180"/>
+<attribute name="BOM" value="EXCLUDE" x="40.64" y="3.81" size="1.778" layer="27" rot="R180" display="off"/>
 </element>
 <element name="P5" library="SparkFun-Connectors" package="1X03_LONGPADS" value="" x="31.75" y="3.81" smashed="yes" rot="R180">
 <attribute name="NAME" x="30.5562" y="7.0612" size="1.016" layer="21" font="vector" ratio="10" rot="R180"/>
 <attribute name="VALUE" x="33.02" y="7.62" size="1.27" layer="27" rot="R180"/>
+<attribute name="BOM" value="EXCLUDE" x="31.75" y="3.81" size="1.778" layer="27" rot="R180" display="off"/>
 </element>
 <element name="P4" library="SparkFun-Connectors" package="1X03_LONGPADS" value="" x="22.86" y="3.81" smashed="yes" rot="R180">
 <attribute name="NAME" x="21.7932" y="7.0612" size="1.016" layer="21" font="vector" ratio="10" rot="R180"/>
 <attribute name="VALUE" x="24.13" y="7.62" size="1.27" layer="27" rot="R180"/>
+<attribute name="BOM" value="EXCLUDE" x="22.86" y="3.81" size="1.778" layer="27" rot="R180" display="off"/>
 </element>
 <element name="P9" library="SparkFun-Connectors" package="1X04_LONGPADS" value="" x="57.15" y="26.035" smashed="yes" rot="R270">
 <attribute name="VALUE" x="53.34" y="27.305" size="1.27" layer="27" rot="R270"/>
+<attribute name="PARTNO" value="826631-4" x="57.15" y="26.035" size="1.778" layer="27" rot="R270" display="off"/>
 </element>
 <element name="P3" library="SparkFun-Connectors" package="1X03_LONGPADS" value="" x="17.78" y="38.1" smashed="yes">
 <attribute name="NAME" x="19.1008" y="34.7218" size="1.016" layer="21" font="vector" ratio="10"/>
 <attribute name="VALUE" x="16.51" y="34.29" size="1.27" layer="27"/>
+<attribute name="BOM" value="EXCLUDE" x="17.78" y="38.1" size="1.778" layer="27" display="off"/>
 </element>
 <element name="P2" library="SparkFun-Connectors" package="1X03_LONGPADS" value="" x="26.67" y="38.1" smashed="yes">
 <attribute name="NAME" x="27.8638" y="34.7218" size="1.016" layer="21" font="vector" ratio="10"/>
 <attribute name="VALUE" x="25.4" y="34.29" size="1.27" layer="27"/>
+<attribute name="BOM" value="EXCLUDE" x="26.67" y="38.1" size="1.778" layer="27" display="off"/>
 </element>
 <element name="P1" library="SparkFun-Connectors" package="1X03_LONGPADS" value="" x="35.56" y="38.1" smashed="yes">
 <attribute name="NAME" x="37.0078" y="34.7218" size="1.016" layer="21" font="vector" ratio="10"/>
 <attribute name="VALUE" x="34.29" y="34.29" size="1.27" layer="27"/>
+<attribute name="BOM" value="EXCLUDE" x="35.56" y="38.1" size="1.778" layer="27" display="off"/>
 </element>
 <element name="LED1" library="adafruit" package="LED3MM" value="" x="55.499" y="10.795" smashed="yes" rot="R270">
 <attribute name="VALUE" x="53.848" y="8.89" size="1.27" layer="27" ratio="10" rot="R270"/>
+<attribute name="PARTNO" value="WP7113SRD/D" x="55.499" y="10.795" size="1.778" layer="27" rot="R270" display="off"/>
 </element>
-<element name="R1" library="resistor" package="0204/7" value="500Ohm" x="58.928" y="10.795" smashed="yes" rot="R270">
+<element name="R1" library="resistor" package="0204/7" value="470Ohm" x="58.928" y="10.795" smashed="yes" rot="R270">
 <attribute name="VALUE" x="58.4454" y="12.4206" size="0.9906" layer="27" ratio="10" rot="R270"/>
+<attribute name="PARTNO" value="CFR-25JR-52-470R" x="58.928" y="10.795" size="1.778" layer="27" rot="R270" display="off"/>
 </element>
 <element name="U1" library="random" package="DIL16" value="MIC5891" x="21.59" y="22.86" smashed="yes" rot="R90">
 <attribute name="NAME" x="26.543" y="12.573" size="1.016" layer="21" font="vector" ratio="10" rot="R180"/>
 <attribute name="VALUE" x="22.225" y="15.367" size="1.27" layer="27" ratio="10" rot="R90"/>
+<attribute name="PARTNO" value="MIC5891YN" x="21.59" y="22.86" size="1.778" layer="27" rot="R90" display="off"/>
 </element>
 <element name="U2" library="random" package="DIL16" value="MIC5891" x="34.036" y="18.288" smashed="yes" rot="R270">
 <attribute name="NAME" x="31.242" y="29.591" size="1.016" layer="21" font="vector" ratio="10" rot="R180"/>
 <attribute name="VALUE" x="33.401" y="25.781" size="1.27" layer="27" ratio="10" rot="R270"/>
+<attribute name="PARTNO" value="MIC5891YN" x="34.036" y="18.288" size="1.778" layer="27" rot="R270" display="off"/>
 </element>
 <element name="U3" library="SparkFun-DigitalIC" package="DIL16" value="HEX_CONVERTERDIP16" x="47.752" y="18.288" smashed="yes" rot="R270">
 <attribute name="NAME" x="43.053" y="28.575" size="1.016" layer="21" font="vector" ratio="10"/>
 <attribute name="VALUE" x="47.117" y="25.781" size="1.27" layer="27" ratio="10" rot="R270"/>
+<attribute name="PARTNO" value="CD74HC4050E" x="47.752" y="18.288" size="1.778" layer="27" rot="R270" display="off"/>
 </element>
 <element name="C4" library="adafruit" package="E7,5-16" value="2000uF" x="8.89" y="9.144" smashed="yes" rot="R270">
 <attribute name="VALUE" x="4.5974" y="14.224" size="1.778" layer="27" ratio="10" rot="R270"/>
+<attribute name="PARTNO" value="EEU-TP1E202S" x="8.89" y="9.144" size="1.778" layer="27" rot="R270" display="off"/>
 </element>
 </elements>
